File: snail-bot/snail-bot.kicad_pcb (KiCad board)
At the start: 2 copper layers, 76 x 24 mm, 50 parts, among them J1 Conn_01x02, J10 Conn_01x02, J11 Conn_01x02, J12 Conn_01x02, J13 Conn_01x02, J2 Conn_01x02, J3 Conn_01x02, J4 TYPE-C-31-M-12, J6 Conn_01x04, J7 Conn_01x02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

Commit message: Add 3D models
Parts:
- J4: footprint snapeda:HRO_TYPE-C-31-M-12 -> homebrew:HRO_TYPE-C-31-M-12
